Commit message: omni urdf updated

File: Week 5/geomagic_ros/omni_description/urdf/omni.urdf (robot description, URDF)
Before this commit: robot phantom_omni, 7 links, 6 joints
Joints:
- joint m1: origin xyz=0 0 0.09 rpy=0 0 0 -> xyz=0 0 0.09 rpy=0 0 3.14159265359
- joint m6: origin xyz=0 -0.023 0 rpy=3.14159 3.14159 0 -> xyz=0 0 0 rpy=3.14159 3.14159 0

Commit message: urdf conf

File: Week 5/geomagic_ros/omni_description/urdf/omni.urdf (robot description, URDF)
Before this commit: robot phantom_omni, 7 links, 6 joints
Joints:
- joint m6: axis 0 1 0 -> 0 0 1; origin xyz=0 0 0 rpy=3.14159 3.14159 0 -> xyz=0 0 0 rpy=1.5707 -1.5707 0
